Commit message: fulll ros1 traduction

File: urdf/arm.urdf (robot description, URDF)
Before this commit: robot dyamixel_arm, 8 links, 7 joints
Links:
- link link2: geometry collision mesh filename=package://dynamixel_arm_description/meshes/chain_link2.stl scale=0.001 0.001 0.001; visual mesh filename=package://dynamixel_arm_description/meshes/chain_link2.stl scale=0.001 0.001 0.001

File: urdf/arm.urdf.xacro (robot description, xacro)
@@ -40,5 +40,5 @@
       <origin xyz="0 0 0.019" rpy="0 0 0"/>
       <geometry>
-        <mesh filename="package://odynamixel_arm_description/meshes/chain_link2.stl" scale="0.001 0.001 0.001"/>
+        <mesh filename="package://dynamixel_arm_description/meshes/chain_link2.stl" scale="0.001 0.001 0.001"/>
       </geometry>
       <material name="blue">
